File: PICTEMPNET.kicad_sch (KiCad schematic)
At the start: 74 parts, among them J1 Barrel Jack, J2 08B0-1X1T-36-F, J3 RJ-12, J4 LCM-S01602DTR_M, SW1 SW_Push, U1 PIC18F97J60-IPT, U2 LM2940S-5.0/NOPB, U3 TC1262-3.3, U4 ENC28J60x-ML, U5 TC1047xNB, Y1 25 MHz, Y2 32 kHz, Y3 25 MHz

Commit message: KiCAD files
Connections:
- net NC0: no longer names the net of J4.15 (LED+)
- net NC1: no longer names the net of J4.16 (LED-)
- no-connect marks 0 -> 54
Other:
- moved on the sheet: C13, C14, C15, C16, C17, C18, C19, D2, J1, R18, R19, R4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
